File: Hardware/D1ZIG.sch (EAGLE design)
At the start: 5 parts

Commit message: Final DRC and tweaks for v1.0 release
Parts:
- removed J3, J4: (no value), freetronics-original:M08
- added J1, J2: (no value), freetronics-original:M08
Connections:
- removed net RX: J4.2
- removed net TX: J4.1
- net 3.3V: now also J1.8; no longer J3.8
- net D1_CC_RST: now also J2.3; no longer J4.3
- net D2_P2_2_DC: now also J2.4; no longer J4.4
- net D6_P2_1_DD: now also J1.5; no longer J3.5
- net D7_P0_3: now also J1.6; no longer J3.6
- net D8_P0_2: now also J1.7; no longer J3.7
- net GND: now also J2.7; no longer J4.7
Other:
- note added: "(C)2020 SuperHouse Automation Pty Ltd: www.superhouse.tv"
- note added: "D1 Mini Zigbee Shield"
- note added: "Licensed under the TAPR Open Hardware License: www.tapr.org/ohl"
- note added: "Power LED"
- note added: "V1.0 (2020-08-15)"
- note removed: "D1Mini Zigbee Shield"
- note removed: "Power"
- note removed: "V1.0 (2020-08-14)"
- moved on the sheet: LED1, MOD1, R1

Commit message: Flipped entire board for reverse mounting on D1 Mini for v1.0 release
Parts:
- R1: value 2K2 -> 4K7
Changed lines of the file:
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@@
 <part name="U$26" library="SuperHouse-SupplySymbols" library_urn="urn:adsk.eagle:library:11790503" deviceset="NC" device=""/>
 <part name="LED1" library="SuperHouse-LEDs" library_urn="urn:adsk.eagle:library:11790571" deviceset="LED" device="0603" package3d_urn="urn:adsk.eagle:package:7066240/3" value="BLUE"/>
-<part name="R1" library="SuperHouse-DiscreteSemi" library_urn="urn:adsk.eagle:library:11768461" deviceset="RESISTOR" device="0603" package3d_urn="urn:adsk.eagle:package:11768543/2" value="2K2"/>
+<part name="R1" library="SuperHouse-DiscreteSemi" library_urn="urn:adsk.eagle:library:11768461" deviceset="RESISTOR" device="0603" package3d_urn="urn:adsk.eagle:package:11768543/2" value="4K7"/>
 <part name="P+1" library="SuperHouse-SupplySymbols" library_urn="urn:adsk.eagle:library:11790503" deviceset="3.3V" device=""/>
 <part name="GND4" library="freetronics-original" deviceset="GND" device=""/>
-<part name="MOD1" library="SuperHouse-Modules" library_urn="urn:adsk.eagle:library:11876743" deviceset="E18-MS1PA" device="" package3d_urn="urn:adsk.eagle:package:22620078/5"/>
+<part name="MOD1" library="SuperHouse-Modules" library_urn="urn:adsk.eagle:library:11876743" deviceset="E18-MS1PA" device="" package3d_urn="urn:adsk.eagle:package:22620078/6"/>
 <part name="GND5" library="freetronics-original" deviceset="GND" device=""/>
 <part name="P+4" library="SuperHouse-SupplySymbols" library_urn="urn:adsk.eagle:library:11790503" deviceset="3.3V" device=""/>
